File: StrainGaugeAmplifier/StrainGaugeAmplifier.sch (KiCad schematic (older format))
At the start: 38 parts, among them K1 BS-115C-12A-12VDC, X1 WF-4, X2 WF-5, X3 WF-6, X4 WF-3

Commit message: Расположил элементы на плате и повёл трассировку.
Parts:
- R10, R12, R17: footprint IWcomponents:RESISTOR_0.25W -> IWcomponents:Electron_3296W
Connections:
- wire segments 143 -> 146
Changed lines of the file:
@@
 	-1   0    0    -1
 $EndComp
-Text Notes 2920 3390 0    50   ~ 0
+Text Notes 2920 3490 0    50   ~ 0
 IN+
-Text Notes 2920 3490 0    50   ~ 0
-IN-
 Text Notes 2890 3590 0    50   ~ 0
 +VCC
@@
 Rk
 Wire Wire Line
-	3500 3350 3950 3350
-Wire Wire Line
 	4300 3550 4200 3550
 Wire Wire Line
 	4200 3550 4200 3450
-Wire Wire Line
-	4200 3450 3500 3450
 Wire Wire Line
 	3500 3550 3850 3550
@@
 F 0 "R10" H 8375 3063 71  0000 C CNN
 F 1 "50 к" H 8375 2940 71  0000 C CNN
-F 2 "IWcomponents:RESISTOR_0.25W" H 8250 2700 60  0001 C CNN
+F 2 "IWcomponents:Electron_3296W" H 8250 2700 60  0001 C CNN
 F 3 "~" H 8375 2931 60  0000 C CNN
 	1    8250 2700
@@
 F 0 "R17" H 11575 3013 71  0000 C CNN
 F 1 "10 к" H 11575 2890 71  0000 C CNN
-F 2 "IWcomponents:RESISTOR_0.25W" H 11450 2650 60  0001 C CNN
+F 2 "IWcomponents:Electron_3296W" H 11450 2650 60  0001 C CNN
 F 3 "~" H 11575 2881 60  0000 C CNN
 	1    11450 2650
@@
 	12050 2650 12050 3150
 Wire Wire Line
-	12050 3350 11950 3350
-Wire Wire Line
 	11950 3150 12050 3150
 Connection ~ 12050 3150
-Wire Wire Line
-	12050 3150 12050 3350
 Wire Wire Line
 	11700 2550 11800 2550
@@
 F 0 "R12" V 9413 2228 71  0000 L CNN
 F 1 "10 к" V 9536 2228 71  0000 L CNN
-F 2 "IWcomponents:RESISTOR_0.25W" H 9350 2050 60  0001 C CNN
+F 2 "IWcomponents:Electron_3296W" H 9350 2050 60  0001 C CNN
 F 3 "~" H 9475 2281 60  0000 C CNN
 	1    9350 2050
@@
 Wire Wire Line
 	10000 4300 13100 4300
-Wire Wire Line
-	13100 4300 13100 3250
-Wire Wire Line
-	13100 3250 13400 3250
 Connection ~ 9350 3150
 Wire Wire Line
@@
 Wire Wire Line
 	4250 4800 4050 4800
-Connection ~ 3950 3350
 Wire Wire Line
 	3950 3350 4300 3350
@@
 Wire Wire Line
 	3500 6750 4000 6750
+Wire Wire Line
+	13100 3250 13400 3250
+Wire Wire Line
+	13100 3250 13100 4300
+Wire Wire Line
+	3500 3350 3750 3350
+Wire Wire Line
+	3750 3350 3750 3450
+Wire Wire Line
+	3750 3450 4200 3450
+Wire Wire Line
+	3500 3450 3650 3450
+Wire Wire Line
+	3650 3450 3650 3250
+Wire Wire Line
+	3650 3250 3950 3250
+Wire Wire Line
+	3950 3250 3950 3350
+Connection ~ 3950 3350
+Text Notes 2920 3390 0    50   ~ 0
+IN-
 $EndSCHEMATC

Commit message: Отправил печатные платы в производство.
Connections:
- wire segments 146 -> 150
Other:
- note added: "Усил. 100"
- note added: "Усил. 30"
Changed lines of the file:
@@
 Wire Wire Line
 	5200 7400 5200 7650
-Text Notes 2860 6880 0    50   ~ 0
+Text Notes 2860 6990 0    50   ~ 0
 +VCC
-Wire Wire Line
-	3500 6850 3600 6850
-Wire Wire Line
-	3600 6850 3600 6650
 Connection ~ 3600 6650
 Wire Wire Line
 	3600 6650 3850 6650
-Text Notes 2790 6990 0    50   ~ 0
+Text Notes 2790 7090 0    50   ~ 0
 RELEY_ON
 $Comp
@@
 	4300 6950 4650 6950
 Wire Wire Line
-	4000 6950 3500 6950
-Wire Wire Line
 	3500 6750 4000 6750
 Wire Wire Line
@@
 Text Notes 2920 3390 0    50   ~ 0
 IN-
+Text Notes 2900 7190 0    50   ~ 0
+GND
+Text Notes 2900 6890 0    50   ~ 0
+GND
+Wire Wire Line
+	3500 6950 3600 6950
+Wire Wire Line
+	3600 6650 3600 6950
+Wire Wire Line
+	3500 6850 3850 6850
+Text Label 3850 7150 2    50   ~ 0
+GND
+Text Label 3850 6850 2    50   ~ 0
+GND
+Wire Wire Line
+	3500 7150 3850 7150
+Wire Wire Line
+	3500 7050 3700 7050
+Wire Wire Line
+	3700 7050 3700 6950
+Wire Wire Line
+	3700 6950 4000 6950
+Text Notes 13830 3390 0    50   ~ 0
+GND
+Text Notes 13760 3290 0    50   ~ 0
+Усил. 30
+Text Notes 13730 3190 0    50   ~ 0
+Усил. 100
 $EndSCHEMATC
