File: Power_supply/Power_supply.sch (KiCad schematic (older format))
At the start: 15 parts, among them X1 DG301-5.0-02P, X2 DG301-5.0-03P

Commit message: Поправил ошибки в схеме и на печатной плате Power_supply.
Connections:
- net -15V: now also DA2.3 (Vout); no longer DA2.2 (Vin)
- net at C2.2, VD1.1, VD2.1: now also DA2.2 (Vin); no longer DA2.3 (Vout)
Changed lines of the file:
@@
 L LFcomponents:7915 DA2
 U 1 1 6231A3E4
-P 6650 4600
-F 0 "DA2" H 6900 4681 60  0000 C CNN
-F 1 "LM7915" H 6900 4787 60  0000 C CNN
-F 2 "IWcomponents:TO220_RAD_16.5x15" H 6650 4600 60  0001 C CNN
-F 3 "" H 6650 4600 60  0000 C CNN
-	1    6650 4600
-	-1   0    0    1
+P 6150 4600
+F 0 "DA2" H 6400 4681 60  0000 C CNN
+F 1 "LM7915" H 6400 4787 60  0000 C CNN
+F 2 "IWcomponents:TO220_RAD_16.5x15" H 6150 4600 60  0001 C CNN
+F 3 "" H 6150 4600 60  0000 C CNN
+	1    6150 4600
+	1    0    0    1
 $EndComp
 Wire Wire Line
